File: PCB_OnlyServo.kicad_sch (KiCad schematic)
At the start: 7 parts, among them J1 Joystick, U1 ICS, U2 R-78E5.0-1.0, U3 SeeeduinoXIAO

Commit message: Add footprint
Parts:
- D1, D2: footprint (none) -> Diode_THT:D_A-405_P10.16mm_Horizontal
- J1: footprint (none) -> Connector_JST:JST_XH_S4B-XH-A_1x04_P2.50mm_Horizontal
- OFFSET1: footprint (none) -> 3386K:3386K
- U1: footprint (none) -> ICS:ICS
- U3: footprint (none) -> Seeeduino XIAO KICAD:Seeeduino XIAO-MOUDLE14P-2.54-21X17.8MM
Changed lines of the file:
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@@
       (effects (font (size 1.27 1.27)))
     )
-    (property "Footprint" "" (at 63.5 41.91 0)
+    (property "Footprint" "Diode_THT:D_A-405_P10.16mm_Horizontal" (at 63.5 41.91 0)
       (effects (font (size 1.27 1.27)) hide)
     )
@@
       (effects (font (size 1.27 1.27)) (justify left))
     )
-    (property "Footprint" "" (at 135.89 55.245 0)
+    (property "Footprint" "Seeeduino XIAO KICAD:Seeeduino XIAO-MOUDLE14P-2.54-21X17.8MM" (at 135.89 55.245 0)
       (effects (font (size 1.27 1.27)) hide)
     )
@@
       (effects (font (size 1.27 1.27)))
     )
-    (property "Footprint" "" (at 73.66 85.725 0)
+    (property "Footprint" "Connector_JST:JST_XH_S4B-XH-A_1x04_P2.50mm_Horizontal" (at 73.66 85.725 0)
       (effects (font (size 1.27 1.27)) hide)
     )
@@
       (effects (font (size 1.27 1.27)))
     )
-    (property "Footprint" "" (at 39.37 38.1 0)
+    (property "Footprint" "ICS:ICS" (at 39.37 38.1 0)
       (effects (font (size 1.27 1.27)) hide)
     )
@@
       (effects (font (size 1.27 1.27)))
     )
-    (property "Footprint" "" (at 93.345 41.91 0)
+    (property "Footprint" "Diode_THT:D_A-405_P10.16mm_Horizontal" (at 93.345 41.91 0)
       (effects (font (size 1.27 1.27)) hide)
     )
@@
       (effects (font (size 1.27 1.27)) (justify right))
     )
-    (property "Footprint" "" (at 107.315 56.515 0)
-      (effects (font (size 1.27 1.27)) hide)
-    )
+    (property "Footprint" "3386K:3386K" (at 107.315 56.515 0)
+      (effects (font (size 1.27 1.27)) hide)
+    )
